File: Switchwire_lightbars/Switchwire_lightbars.kicad_pcb (KiCad board)
At the start: 2 copper layers, 35 x 15.2 mm, 3 parts, among them J1 Conn_01x03_Male

Commit message: Another few changes
Another few changes
Parts:
- added C10: 0.1uF, Capacitor_SMD:C_0805_2012Metric, F.Cu at (44.3, 58.5)
- added C11: 0.1uF, Capacitor_SMD:C_0805_2012Metric, F.Cu at (47.5, 54.8)
- added C12: 0.1uF, Capacitor_SMD:C_0805_2012Metric, F.Cu at (52.0, 51.9)
- added C13: 0.1uF, Capacitor_SMD:C_0805_2012Metric, F.Cu at (56.0, 48.2)
- added C2: 0.1uF, Capacitor_SMD:C_0805_2012Metric, F.Cu at (48.8, 57.8)
- added C3: 0.1uF, Capacitor_SMD:C_0805_2012Metric, F.Cu at (22.3, 58.5)
- added C4: 0.1uF, Capacitor_SMD:C_0805_2012Metric, F.Cu at (26.7, 58.5)
- added C5: 0.1uF, Capacitor_SMD:C_0805_2012Metric, F.Cu at (31.1, 58.5)
- added C6: 0.1uF, Capacitor_SMD:C_0805_2012Metric, F.Cu at (35.5, 58.5)
- added C7: 0.1uF, Capacitor_SMD:C_0805_2012Metric, F.Cu at (47.5, 51.9)
- added C8: 0.1uF, Capacitor_SMD:C_0805_2012Metric, F.Cu at (39.9, 58.5)
- added C9: 0.1uF, Capacitor_SMD:C_0805_2012Metric, F.Cu at (56.0, 45.2)
- added D10: WS2812B, LED_SMD:LED_WS2812B_PLCC4_5.0x5.0mm_P3.2mm, F.Cu at (41.1, 53.7)
- added D11: WS2812B, LED_SMD:LED_WS2812B_PLCC4_5.0x5.0mm_P3.2mm, F.Cu at (49.6, 47.1)
- added D12: WS2812B, LED_SMD:LED_WS2812B_PLCC4_5.0x5.0mm_P3.2mm, F.Cu at (58.0, 40.4)
- added D13: WS2812B, LED_SMD:LED_WS2812B_PLCC4_5.0x5.0mm_P3.2mm, F.Cu at (24.3, 40.4)
- added D2: WS2812B, LED_SMD:LED_WS2812B_PLCC4_5.0x5.0mm_P3.2mm, F.Cu at (24.3, 47.1)
- added D3: WS2812B, LED_SMD:LED_WS2812B_PLCC4_5.0x5.0mm_P3.2mm, F.Cu at (32.7, 40.4)
- added D4: WS2812B, LED_SMD:LED_WS2812B_PLCC4_5.0x5.0mm_P3.2mm, F.Cu at (24.3, 53.7)
- added D5: WS2812B, LED_SMD:LED_WS2812B_PLCC4_5.0x5.0mm_P3.2mm, F.Cu at (32.7, 47.1)
- added D6: WS2812B, LED_SMD:LED_WS2812B_PLCC4_5.0x5.0mm_P3.2mm, F.Cu at (41.1, 40.4)
- added D7: WS2812B, LED_SMD:LED_WS2812B_PLCC4_5.0x5.0mm_P3.2mm, F.Cu at (32.7, 53.7)
- added D8: WS2812B, LED_SMD:LED_WS2812B_PLCC4_5.0x5.0mm_P3.2mm, F.Cu at (41.1, 47.1)
- added D9: WS2812B, LED_SMD:LED_WS2812B_PLCC4_5.0x5.0mm_P3.2mm, F.Cu at (49.6, 40.4)
- J1: footprint Connector_JST:JST_XH_S3B-XH-A_1x03_P2.50mm_Horizontal -> Connector_JST:JST_SUR_SM03B-SURS-TF_1x03-1MP_P0.80mm_Horizontal
- moved J1 9.23 mm to (23.2, 26.5)
Connections:
- D1 pad 2: 1out -> Net-(D1-Pad2)
Routing:
- removed copper zone on F.Cu, net +5V
- removed copper zone on B.Cu, net GND
- removed copper zone on F.Cu, net GND
Other:
- board size 35 x 15.2 mm -> 238 x 10 mm
